File: PCB/GPS_PCB/GPS_PCB.kicad_sch (KiCad schematic)
At the start: 0 parts

Commit message: Update
Parts:
- added C120: 10uF, Capacitor_SMD:C_1206_3216Metric, symbol Device:C
- added C79, C80: 0.1uF, Capacitor_SMD:C_0603_1608Metric, symbol Device:C
- added FPC1: FPC-05F-6PH20, lcsc:FPC-SMD_6P-P0.50_XUNPU_FPC-05F-6PH20, symbol LCSC:FPC-05F-6PH20
- added R1: 4.7K, Resistor_SMD:R_0603_1608Metric, symbol Device:R
- added U1: CR2032-BS-6, lcsc:BAT-TH_CR2032-BS-6-1, symbol LCSC:CR2032-BS-6
- added U26: L80RE-M37, lcsc:GPSM-SMD_12P-L16.0-W16.0-P2.54-BL, symbol LCSC:L80RE-M37
Connections:
- new net: C79.2, U1.1, U26.5 (V_BCKP)
- new net +3.3V: C120.2, C80.2, FPC1.5, FPC1.6, R1.1, U26.4 (VCC)
- new net GND: C120.1, C79.1, C80.1, FPC1.3, FPC1.4, FPC1.7, FPC1.8, U1.2, U26.12 (GND), U26.3 (GND)
- new net GPS_RX: FPC1.1, U26.1 (RXD1)
- new net GPS_TX: FPC1.2, U26.2 (TXD1)
- new net Reset: R1.2, U26.10 (RESET)
- no-connect marks 0 -> 5
Other:
- note added: "GPS"
